Commit message: final

File: path_planning_ws/src/maze_bot/urdf/maze_bot.urdf (robot description, URDF)
Before this commit: robot maze_bot, 6 links, 5 joints
Links:
- added link top_marker_link, mass 0.03; collision cylinder length=0.10 radius=0.02; visual cylinder length=0.10 radius=0.02
- link camera_link: mass None -> 0.05; geometry collision box size=0.03 0.03 0.02; visual box size=0.03 0.03 0.02
Joints:
- added joint top_marker_joint: type fixed, parent base, child top_marker_link, origin xyz=0.0 0.0 0.20 rpy=0 0 0
